File: Stikka-Controller.kicad_pcb (KiCad board)
At the start: 2 copper layers, 42 x 23 mm, 36 parts, among them J1 Conn_01x02_Socket, J2 Conn_01x02_Socket, J3 Conn_01x02_Socket, J4 Conn_01x05_Socket, J6 Conn_01x03_Socket, J7 GROVE-CONNECTOR-SMD-90D_4+2P-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, Q1 SS8050, Q2 SS8050, U1 ESP32-S3-WROOM-1, U2 AP2127N-3.3, U5 RBT10W24S05

Commit message: moved some parts
Parts:
- added kibuzzard-6A99DAF3: G***, kibuzzard-6A99DAF3, F.Cu at (158.1, 104.8)
- added kibuzzard-6A99DAF3: G***, kibuzzard-6A99DAF3, B.Cu at (158.1, 104.8)
- added kibuzzard-6A99DB3D: G***, kibuzzard-6A99DB3D, F.Cu at (158.1, 102.3)
- added kibuzzard-6A99DB3D: G***, kibuzzard-6A99DB3D, B.Cu at (158.1, 102.3)
- added kibuzzard-6A99DB6C: G***, kibuzzard-6A99DB6C, F.Cu at (158.1, 107.3)
- added kibuzzard-6A99DB6C: G***, kibuzzard-6A99DB6C, B.Cu at (158.1, 107.3)
- added kibuzzard-6A9B1D11: G***, kibuzzard-6A9B1D11, B.Cu at (127.0, 105.3)
- added kobee-studio-6A9B380E: Kobee Studio, kobee-studio-6A9B380E, B.Cu at (145.2, 107.1)
- moved J3 52.3 mm to (159.2, 114.5)
- moved kibuzzard-6A99DAF3 52.3 mm to (155.6, 115.4)
- moved kibuzzard-6A99DB3D 52.3 mm to (155.6, 113.6)
- moved kibuzzard-6A99E40F 52.3 mm to (157.3, 117.0)
- moved U5 50.4 mm to (154.4, 102.3)
- moved Q2 49.8 mm to (141.5, 112.1)
- moved R2 49.8 mm to (141.5, 115.1)
- moved J4 49.8 mm to (148.7, 120.2)
- moved J7 49.8 mm to (145.0, 103.4)
- moved R1 49.8 mm to (144.5, 117.2)
- moved kibuzzard-6A99DCAC 49.8 mm to (148.7, 117.0)
- moved kibuzzard-6A99DCB6 49.8 mm to (153.7, 117.0)
- moved C1 49.8 mm to (128.6, 120.4)
- moved C11 49.8 mm to (120.8, 120.4)
- moved C12 49.8 mm to (124.7, 120.4)
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Routing:
- net GND: track 48.3 -> 62.2 mm, vias 78 -> 92
- net +5V: track 28.3 -> 38.4 mm
- net /LED: track 10.5 -> 3.35 mm
- net /BOOT: track 19.1 -> 25.3 mm, vias 2 -> 1
- net VIN: track 15.1 -> 16.2 mm
- net /RST: track 41.0 -> 40.7 mm, vias 4 -> 3
